File: prj/WifiRemote.sch (KiCad schematic (older format))
At the start: 9 parts, among them K1 DIP-SWITCH-TACTILE-SPST-NO_TS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, K2 DIP-SWITCH-TACTILE-SPST-NO_TS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, K3 DIP-SWITCH-TACTILE-SPST-NO_TS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, K4 DIP-SWITCH-TACTILE-SPST-NO_TS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, U1 PMIC-MP1496DJ_SOT23-8_

Commit message: Completed power supply design
Parts:
- added C1: CERAMIC-22UF-25V-20%-X5R_0805_, symbol CERAMIC-22UF-25V-20%-X5R_0805_
- added C2: CERAMIC-100NF-50V-10%-X7R_0603_, symbol CERAMIC-100NF-50V-10%-X7R_0603_
- added C3: CERAMIC-22NF-50V-10%-X7R_0603_, symbol CERAMIC-22NF-50V-10%-X7R_0603_
- added C5: CERAMIC-47UF-10V-20%-X5R_0805_, symbol CERAMIC-47UF-10V-20%-X5R_0805_
- added D1, D2: SMD-RGB-LED-4P, symbol SMD-RGB-LED-4P
- added L1: SMD-INDUCTOR-5.6UH-30%-1.64A, symbol SMD-INDUCTOR-5.6UH-30%-1.64A
- added R1: SMD-RES-30K-1%-1_10W_0603_, symbol SMD-RES-30K-1%-1_10W_0603_
- added R3: SMD-RES-33K-1%-1_10W_0603_, symbol SMD-RES-33K-1%-1_10W_0603_
- added R4: SMD-RES-40.2K-1%-1_10W_0603_, symbol SMD-RES-40.2K-1%-1_10W_0603_
- added R5: SMD-RES-13K-1%-1_10W_0603_, symbol SMD-RES-13K-1%-1_10W_0603_
- renumbered C1 to C4, D1 to D3, D2 to D4, K3 to K2, K2 to K3, R1 to R2
Connections:
- net labels added: +3.3V, +BATT
- wire segments 4 -> 13
Other:
- moved on the sheet: C4, K1, K2, K3, K4, R2

Commit message: Added ESP and FTDI interface in Schematic
Parts:
- removed D3, D4: SMD-DIODE-TVS-5V-225MW_SOT-23_, symbol SMD-DIODE-TVS-5V-225MW_SOT-23_
- added C6: CERAMIC-10NF-50V-5%-X7R_0805_, symbol CERAMIC-10NF-50V-5%-X7R_0805_
- added D3: SMD-DIODE-SCHOTTKY-40V-1A_DO-214AC_, symbol SMD-DIODE-SCHOTTKY-40V-1A_DO-214AC_
- added J1: DIP-BLACK-MALE-HEADER_6P-2.54_, symbol DIP-BLACK-MALE-HEADER_6P-2.54_
- added R6, R7, R8, R9: SMD-RES-10K-5%-1_10W_0603_, symbol SMD-RES-10K-5%-1_10W_0603_
- added U?: CONTROLLER-ESP8266, symbol CONTROLLER-ESP8266
Connections:
- net labels added: EN, FTDI_DTR, FTDI_RXI, FTDI_TXO, GPIO0, GPIO15, GPIO2
- wire segments 13 -> 25
Other:
- note added: "Need TVS for this Line"
- moved on the sheet: K1, K2

Commit message: Added push buttons, ESP programming lines, and battery voltage monitoring
Parts:
- removed C6: CERAMIC-10NF-50V-5%-X7R_0805_, symbol CERAMIC-10NF-50V-5%-X7R_0805_
- removed D1: SMD-RGB-LED-4P, symbol SMD-RGB-LED-4P
- removed D3: SMD-DIODE-SCHOTTKY-40V-1A_DO-214AC_, symbol SMD-DIODE-SCHOTTKY-40V-1A_DO-214AC_
- removed U?: CONTROLLER-ESP8266, symbol CONTROLLER-ESP8266
- added C6: CERAMIC-100NF-50V-10%-X7R_0805_, symbol CERAMIC-100NF-50V-10%-X7R_0805_
- added D2, D3, D4, D5: SMD-DIODE-SWITCH-1N4148_LL-34_, symbol SMD-DIODE-SWITCH-1N4148_LL-34_
- added D6, D7: SMD-DIODE-SCHOTTKY-20V-500MA_SOD-123_, symbol SMD-DIODE-SCHOTTKY-20V-500MA_SOD-123_
- added R1: SMD-RES-10K-1%-1_10W_0603_, symbol SMD-RES-10K-1%-1_10W_0603_
- added R10, R11, R12, R13, R14, R4, R6: SMD-RES-10K-5%-1_10W_0603_, symbol SMD-RES-10K-5%-1_10W_0603_
- added R2: SMD-RES-1K-1%-1_10W_0603_, symbol SMD-RES-1K-1%-1_10W_0603_
- added U2: CONTROLLER-ESP8266, symbol CONTROLLER-ESP8266
- renumbered D2 to D1, K3 to K2, K2 to K3, R6 to R15, R7 to R16, R8 to R17, R9 to R18, R1 to R3, R2 to R5, R3 to R7, R4 to R8, R5 to R9
Connections:
- net labels added: ESP_ADC, GPIO12, GPIO13, GPIO14, GPIO4, GPIO5
- wire segments 25 -> 61
Other:
- note added: "Bypass Cap?"
- note added: "Need 5V Input... Probably switch to two single colored LEDs"
- note added: "Need TVS on Buttons"
- note added: "Need TVS or Zener for this Line?"
- note removed: "Need TVS for this Line"
- moved on the sheet: C2, C4, K1, K2, K3, K4, R17, R18, R5

Commit message: Added power switch
Parts:
- added SW1: DIP-TOGGLE-SWITCH-ON-ON_3+2P-8.8X4.6MM_-90D, symbol DIP-TOGGLE-SWITCH-ON-ON_3+2P-8.8X4.6MM_-90D
- renumbered R6 to R5, R5 to R6
Connections:
- wire segments 61 -> 43
Other:
- note added: "Need 5V Input... Probably switch to two single colored LED(s)"
- note added: "What is the COM pin?"
- note removed: "Need 5V Input... Probably switch to two single colored LEDs"
- moved on the sheet: C2, C4, D2, D3, D4, D5, D6, D7, J1, K1, K2, K3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

Commit message: Added libraries and several components to schematic
Parts:
- removed C1: CERAMIC-22UF-25V-20%-X5R_0805_, symbol CERAMIC-22UF-25V-20%-X5R_0805_
- removed C2, C4: CERAMIC-100NF-50V-10%-X7R_0603_, symbol CERAMIC-100NF-50V-10%-X7R_0603_
- removed C3: CERAMIC-22NF-50V-10%-X7R_0603_, symbol CERAMIC-22NF-50V-10%-X7R_0603_
- removed C5: CERAMIC-47UF-10V-20%-X5R_0805_, symbol CERAMIC-47UF-10V-20%-X5R_0805_
- removed D1: SMD-RGB-LED-4P, symbol SMD-RGB-LED-4P
- removed L1: SMD-INDUCTOR-5.6UH-30%-1.64A, symbol SMD-INDUCTOR-5.6UH-30%-1.64A
- removed R3: SMD-RES-30K-1%-1_10W_0603_, symbol SMD-RES-30K-1%-1_10W_0603_
- removed R4, R5: SMD-RES-10K-5%-1_10W_0603_, symbol SMD-RES-10K-5%-1_10W_0603_
- removed R6: SMD-RES-10R-5%-1_10W_0603_, symbol SMD-RES-10R-5%-1_10W_0603_
- removed R7: SMD-RES-33K-1%-1_10W_0603_, symbol SMD-RES-33K-1%-1_10W_0603_
- removed R8: SMD-RES-40.2K-1%-1_10W_0603_, symbol SMD-RES-40.2K-1%-1_10W_0603_
- removed R9: SMD-RES-13K-1%-1_10W_0603_, symbol SMD-RES-13K-1%-1_10W_0603_
- removed SW1: DIP-TOGGLE-SWITCH-ON-ON_3+2P-8.8X4.6MM_-90D, symbol DIP-TOGGLE-SWITCH-ON-ON_3+2P-8.8X4.6MM_-90D
- removed U1: PMIC-MP1496DJ_SOT23-8_, symbol PMIC-MP1496DJ_SOT23-8_
- added D?: SMD-LED-CLEAR-GREEN_0805_, symbol SMD-LED-CLEAR-GREEN_0805_
- added R?: SMD-RES-10R-5%-1_10W_0603_, symbol SMD-RES-10R-5%-1_10W_0603_
- added U?: PMIC-ETA3410D2I-T_DFN8-2X2_, symbol PMIC-ETA3410D2I-T_DFN8-2X2_
Connections:
- wire segments 43 -> 26
Other:
- note removed: "What is the COM pin?"

Commit message: Added inductors library and wired boost regulator
Parts:
- removed U?: PMIC-ETA3410D2I-T_DFN8-2X2_, symbol PMIC-ETA3410D2I-T_DFN8-2X2_
- added C?: CERAMIC-4.7UF-10V-10%-X5R_0603_, symbol CERAMIC-4.7UF-10V-10%-X5R_0603_
- added C? (x2): CERAMIC-22UF-6.3V-20%-X5R_0805_, symbol CERAMIC-22UF-6.3V-20%-X5R_0805_
- added L?: SMD-Inductor-4.7uH-20%-L0420, symbol SMD-Inductor-4.7uH-20%-L0420
- added R?: SMD-RES-150K-1%-1_10W_0603_, symbol SMD-RES-150K-1%-1_10W_0603_
- added R?: SMD-RES-261K-1%-1_10W_0603_, symbol SMD-RES-261K-1%-1_10W_0603_
- added R? (x2): SMD-RES-0R-5%-1_10W_0603_, symbol SMD-RES-0R-5%-1_10W_0603_
- added R? (x2): SMD-RES-10K-1%-1_10W_0603_, symbol SMD-RES-10K-1%-1_10W_0603_
- added U?: BOOST-MCP1642B-ADJI/MC-MSOP8, symbol BOOST-MCP1642B-ADJI/MC-MSOP8
- R1: RESISTANCE (none) -> 10K
Connections:
- net labels added: 3V3_OUT, GNDD
- wire segments 26 -> 54

Commit message: Rev1 schematic all components placed and wired
Parts:
- removed C6: CERAMIC-100NF-50V-10%-X7R_0805_, symbol CERAMIC-100NF-50V-10%-X7R_0805_
- removed D6: SMD-DIODE-SCHOTTKY-20V-500MA_SOD-123_, symbol SMD-DIODE-SCHOTTKY-20V-500MA_SOD-123_
- removed R16: SMD-RES-10K-5%-1_10W_0603_, symbol SMD-RES-10K-5%-1_10W_0603_
- added C1: CERAMIC-1UF-25V-10%-X7R_0603_, symbol CERAMIC-1UF-25V-10%-X7R_0603_
- added C5: CERAMIC-10UF-10V-10%-X5R_0603_, symbol CERAMIC-10UF-10V-10%-X5R_0603_
- added D10, D12, D6, D8: SMD-Diode-TVS-3.3VMW-15V-SOD-523, symbol SMD-Diode-TVS-3.3VMW-15V-SOD-523
- added D2: SMD-DIODE-SCHOTTKY-20V-500MA_SOD-123_, symbol SMD-DIODE-SCHOTTKY-20V-500MA_SOD-123_
- added D3: SMD-LED-CLEAR-GREEN_0805_, symbol SMD-LED-CLEAR-GREEN_0805_
- added J1: DIP-BLACK-MALE-HEADER-VERT_4P-2.54_, symbol DIP-BLACK-MALE-HEADER-VERT_4P-2.54_
- added R10, R6: SMD-RES-10K-5%-1_10W_0603_, symbol SMD-RES-10K-5%-1_10W_0603_
- added R15, R3, R4, R7: SMD-RES-0R-5%-1_10W_0603_, symbol SMD-RES-0R-5%-1_10W_0603_
- added R23: SMD-RES-10R-5%-1_10W_0603_, symbol SMD-RES-10R-5%-1_10W_0603_
- added SW1: DIP-TOGGLE-SWITCH-ON-ON_3+2P-8.8X4.6MM_-90D, symbol DIP-TOGGLE-SWITCH-ON-ON_3+2P-8.8X4.6MM_-90D
- C4: renamed from C?; PLACE (none) -> DNP
- R1: renamed from R15; RESISTANCE (none) -> 10K
- R12: renamed from R?; RESISTANCE (none) -> 261K; VAL 261K -> (none)
- R16: renamed from R17; RESISTANCE (none) -> 10K
- R17: renamed from R18; RESISTANCE (none) -> 10K
- R18: renamed from R10; RESISTANCE (none) -> 10K
- R19: renamed from R11; RESISTANCE (none) -> 10K
- R20: renamed from R12; RESISTANCE (none) -> 10K
- R21: renamed from R13; RESISTANCE (none) -> 10K
- R22: renamed from R14; RESISTANCE (none) -> 10K
- R24: renamed from R?; RESISTANCE (none) -> 10
- R9: renamed from R2; Resistance (none) -> 1k
- U1: renamed from U2; MANUFACTURER (none) -> -; PART NUMBER (none) -> ESP8266 ESP-12; SKU 310060021 -> (none); SUPPLIER (none) -> ITEAD; SUPPLIER PART (none) -> ESP8266 ESP-12
- gave numbers to parts that had none: 10
- renumbered D7 to D1, D5 to D11, D2 to D5, D3 to D7, D4 to D9, J1 to J2, R1 to R2
Connections:
- net labels added: BTN_INT, ESP_VCC, REG_IN, RST, SW1, SW2, SW3, SW4, SWITCH_BAT
- net labels removed: EN, GND
- wire segments 54 -> 97
- no-connect marks 0 -> 11
Other:
- note removed: "Bypass Cap?"
- note removed: "Need 5V Input... Probably switch to two single colored LED(s)"
- note removed: "Need TVS on Buttons"
- note removed: "Need TVS or Zener for this Line?"
- moved on the sheet: C2, C3, C4, D1, D11, D4, D5, D7, D9, J2, K1, K2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

Commit message: Arranged designators, Added text descriptions, changed border template
Parts:
- added R18: SMD-RES-0R-5%-1_10W_0603_, symbol SMD-RES-0R-5%-1_10W_0603_
- renumbered R11 to R10, R10 to R11, R16 to R15, R15 to R16, R18 to R19, R19 to R20, R20 to R21, R21 to R22, R22 to R23, R23 to R24, R24 to R25
Connections:
- net labels added: BTN_PWR
- wire segments 97 -> 146
Other:
- note added: "PROGRAMMING \nHEADER"
- note added: "SERIAL BOOTLOADER \nENABLE"
- moved on the sheet: C1, C5, D1, D10, D11, D12, D2, D3, D4, D5, D6, D7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
